Commit message: Troubleshooting very annoying orientation issue on the IK solution - stupid rad|degree conversion

File: robotic-arm-control-app/kinematics/urdf/mogarobot.urdf.xacro (robot description, xacro)
@@ -57,4 +57,5 @@
     </link>
     <link name="end_effector_frame"/>
+    <link name="white_gripper_link"/>
     <joint name="world_base_joint" type="fixed">
         <parent link="world"/>
@@ -102,3 +103,8 @@
         <origin xyz="0.2 0 0" rpy="0 0 0"/>
     </joint>
+    <joint name="end_effector_gripper_joint" type="fixed">
+        <parent link="end_effector_frame"/>
+        <child link="white_gripper_link"/>
+        <origin xyz="1.2 0 0" rpy="0 0 0"/>
+    </joint>
 </robot>

Commit message: Added offset to the between the wrist and the hand on the robotic arm to match physical robot

File: robotic-arm-control-app/kinematics/urdf/mogarobot.urdf.xacro (robot description, xacro)
@@ -94,5 +94,5 @@
         <parent link="wrist_link"/>
         <child link="hand_link"/>
-        <origin xyz="0.255 0 0" rpy="0 0 0"/>
+        <origin xyz="0.295 0 0" rpy="0 0 0"/>
         <axis xyz="1 0 0"/>
         <limit lower="-3.14" upper="3.14" effort="30" velocity="10"/>
